File: iium_sumo.kicad_pcb (KiCad board)
At the start: 2 copper layers, 101.3 x 62.2 mm, 58 parts, among them J12 Conn_01x04, J14 Conn_01x04, J15 EXTRA1, J16 Conn_01x02_Pin, J17 Conn_01x02_Pin, SW1 SW_SPST, SW2 SW_SPST, U1 TPS54360DDA, U4 Black Pill v2, U5 LM3940

Commit message: fixed errors
Parts:
- J12, J14: footprint Connector_PinHeader_1.00mm:PinHeader_1x04_P1.00mm_Vertical -> Connector_PinHeader_2.54mm:PinHeader_1x04_P2.54mm_Vertical
- J13: renamed from 5V; footprint Connector_PinHeader_1.00mm:PinHeader_1x04_P1.00mm_Vertical -> Connector_PinHeader_2.54mm:PinHeader_1x04_P2.54mm_Vertical
- moved J14 6.85 mm to (165.2, 76.5)
- moved J13 6.19 mm to (172.8, 72.5)
- moved J16 5.60 mm to (192.7, 106.2), turned to -90 degrees
- moved J17 4.80 mm to (192.3, 97.8), turned to 90 degrees
- moved J12 4.26 mm to (165.2, 68.5)
- moved C13 0.09 mm to (186.6, 98.2)
- renumbered VL53_1 to J1, MD to J10, Cytron_SM to J11, UART1 to J18, UART2 to J19, VL53_2 to J2, VL53_3 to J3, VL53_4 to J4, VL53_5 to J5, IR1 to J6, IR2 to J7, IR3 to J8, IR4 to J9
Routing:
- net GND: track 77.0 -> 49.7 mm, vias 0 -> 68
- net +5V: track 158.1 -> 166.0 mm
- net COMP: track 7.43 -> 12.6 mm
- net FB: track 14.7 -> 11.4 mm
- net +36V: track 30.5 -> 27.4 mm
- net +3V3: track 164.8 -> 167.2 mm, vias 2 -> 3
